Commit message: URDF small objects correctly spwan in RVIZ

File: visualization/urdf/object_black_box_base.urdf.xacro (robot description, xacro)
@@ -24,5 +24,5 @@
       </geometry>
       <material name="black">
-          <color rgba="1 1 1 1"/>
+          <color rgba="0 0 0 1"/>
       </material>
     </visual>

File: visualization/urdf/object_black_cylinder_base.urdf.xacro (robot description, xacro)
@@ -23,6 +23,6 @@
         <cylinder length="0.2" radius="0.15"/>
     </geometry>
-    <material name="blue">
-        <color rgba="0 0 .8 0"/>
+    <material name="black">
+        <color rgba="0 0 0 1"/>
     </material>
   </visual>

File: visualization/urdf/object_blue_box_base.urdf.xacro (robot description, xacro)
@@ -24,5 +24,5 @@
       </geometry>
       <material name="blue">
-          <color rgba="0 0 .8 0"/>
+          <color rgba="0 0 .8 1"/>
       </material>
     </visual>

File: visualization/urdf/object_blue_cylinder_base.urdf.xacro (robot description, xacro)
@@ -24,5 +24,5 @@
       </geometry>
       <material name="blue">
-          <color rgba="0 0 .8 0"/>
+          <color rgba="0 0 .8 1"/>
       </material>
     </visual>

File: visualization/urdf/object_red_box_base.urdf.xacro (robot description, xacro)
@@ -23,6 +23,6 @@
           <box size="0.3 0.3 0.20"/>
       </geometry>
-      <material name="blue">
-          <color rgba="0 0 .8 0"/>
+      <material name="red">
+          <color rgba="0.8 0 0 1"/>
       </material>
     </visual>

File: visualization/urdf/object_red_cylinder_base.urdf.xacro (robot description, xacro)
@@ -23,6 +23,6 @@
           <cylinder length="0.2" radius="0.15"/>
       </geometry>
-      <material name="blue">
-          <color rgba="0 0 .8 0"/>
+      <material name="red">
+          <color rgba="0.8 0 0 1"/>
       </material>
     </visual>
