Commit message: Thursday 7_7

File: visualization/urdf/object_black_cylinder_base.urdf.xacro (robot description, xacro)
@@ -10,34 +10,34 @@
 <xacro:include filename="$(find grvc_quadrotor_gazebo)/urdf/quadrotor_plugins.urdf.xacro" />
 <!--#####################################################################################-->
-  <!-- Main object link -->
-  <xacro:macro name="quadrotor_base_macro" params="id model_name">
-    <link name="base_link_${id}">
-      <inertial>
-        <mass value="0.5" />
-        <origin xyz="0 0 0.0" />
-        <inertia ixx="0.01152" ixy="0.0" ixz="0.0" iyy="0.01152" iyz="0.0" izz="0.0218" />
-      </inertial>
-      <visual>
-      <origin xyz="0 0 0" rpy="0 0 0" />
-      <geometry>
-          <cylinder length="0.2" radius="0.15"/>
-      </geometry>
-      <material name="blue">
-          <color rgba="0 0 .8 0"/>
-      </material>
-    </visual>
-    <collision>
-      <origin xyz="0 0 0" rpy="0 0 0" />
-      <geometry>
-          <cylinder length="0.2" radius="0.15"/>
-      </geometry>
-    </collision>
-  </link>
-    <gazebo reference="base_link_${id}">
-      <material>Gazebo/Black</material>
-      <turnGravityOff>false</turnGravityOff>
-    </gazebo>
-    <!-- Gazebo Plugins -->
-    <xacro:quadrotor_plugins model_name="${model_name}" base_link="base_link_${id}"/>
-  </xacro:macro>
+<!-- Main object link -->
+<xacro:macro name="quadrotor_base_macro" params="id model_name">
+  <link name="base_link_${id}">
+    <inertial>
+      <mass value="0.5" />
+      <origin xyz="0 0 0.0" />
+      <inertia ixx="0.01152" ixy="0.0" ixz="0.0" iyy="0.01152" iyz="0.0" izz="0.0218" />
+    </inertial>
+    <visual>
+    <origin xyz="0 0 0" rpy="0 0 0" />
+    <geometry>
+        <cylinder length="0.2" radius="0.15"/>
+    </geometry>
+    <material name="blue">
+        <color rgba="0 0 .8 0"/>
+    </material>
+  </visual>
+  <collision>
+    <origin xyz="0 0 0" rpy="0 0 0" />
+    <geometry>
+        <cylinder length="0.2" radius="0.15"/>
+    </geometry>
+  </collision>
+</link>
+  <gazebo reference="base_link_${id}">
+    <material>Gazebo/Black</material>
+    <turnGravityOff>false</turnGravityOff>
+  </gazebo>
+  <!-- Gazebo Plugins -->
+  <xacro:quadrotor_plugins model_name="${model_name}" base_link="base_link_${id}"/>
+</xacro:macro>
 </robot>

Commit message: Release object

File: visualization/urdf/object_black_cylinder_base.urdf.xacro (robot description, xacro)
@@ -14,5 +14,5 @@
   <link name="base_link_${id}">
     <inertial>
-      <mass value="0.01" />
+      <mass value="0.5" />
       <origin xyz="0 0 0.0" />
       <inertia ixx="0.01" ixy="0.0" ixz="0.0" iyy="0.01" iyz="0.0" izz="0.01" />

File: visualization/urdf/quadrotor_simple_controller.urdf.xacro (robot description, xacro)
@@ -24,5 +24,5 @@
         <velocityXYProportionalGain>5.0</velocityXYProportionalGain>
         <velocityXYDifferentialGain>1.0</velocityXYDifferentialGain>
-        <velocityXYLimit>5</velocityXYLimit>
+        <velocityXYLimit>50</velocityXYLimit>
         <velocityZProportionalGain>5.0</velocityZProportionalGain>
         <velocityZDifferentialGain>1.0</velocityZDifferentialGain>
