Commit message: Fixed

File: visualization/urdf/grvc_quadrotor_base.urdf.xacro (robot description, xacro)
@@ -50,6 +50,6 @@
     </joint>
   </xacro:macro>
-<!--#####################################################################################-->
-    <!-- Camera -->
+<!--##############################CAMERA#######################################################-->
+  <!-- Camera -->
   <xacro:macro name="generic_camera" params="id">
   	<link name="camera_link_${id}">
@@ -114,4 +114,65 @@
     </gazebo>
   </xacro:macro>
+  <!-- #########################SONAR############################################### -->
+  <xacro:macro name="sonar_sensor" params="id">
+    <link name="sonar_link_${id}">
+      <inertial>
+        <mass value="0.000" />
+        <origin xyz="0 0 0" rpy="0 0 0" />
+        <inertia ixx="0.00000000" ixy="0" ixz="0" iyy="0.00000000" iyz="0" izz="0.00000000" />
+      </inertial>
+      <visual>
+        <origin xyz="0 0 0" rpy="0 0 0" />
+        <geometry>
+          <mesh filename="package://hector_sensors_description/meshes/sonar_sensor/max_sonar_ez4.dae"/>
+        </geometry>
+      </visual>
+      <collision>
+        <origin xyz="0 0 0" rpy="0 0 0" />
+        <geometry>
+          <box size="0.01 0.01 0.01" />
+        </geometry>
+      </collision>
+    </link>
+    <joint name="sonar_${id}_joint" type="fixed">
+      <origin xyz="0 0.25 0.032" rpy="0 1.57 0"/>
+      <parent link="base_link_${id}"/>
+      <child link="sonar_link_${id}"/>
+    </joint>
+    <gazebo reference="sonar_link_${id}">
+      <sensor type="ray" name="sonar_link_${id}_sensor">
+        <always_on>true</always_on>
+        <update_rate>10</update_rate>
+        <pose>0 0 0 0 0 0</pose>
+        <visualize>false</visualize>
+        <ray>
+          <scan>
+            <horizontal>
+              <samples>3</samples>
+              <resolution>1</resolution>
+              <min_angle>-0.35</min_angle>
+              <max_angle> 0.35</max_angle>
+            </horizontal>
+            <vertical>
+              <samples>3</samples>
+              <resolution>1</resolution>
+              <min_angle>-0.35</min_angle>
+              <max_angle>0.35</max_angle>
+            </vertical>
+          </scan>
+          <range>
+            <min>0.03</min>
+            <max>100</max>
+            <resolution>0.01</resolution>
+          </range>
+        </ray>
+        <plugin name="gazebo_ros_sonar_link_${id}_controller" filename="libhector_gazebo_ros_sonar.so">
+          <gaussianNoise>0.005</gaussianNoise>
+          <topicName>sonar_${id}</topicName>
+          <frameId>sonar_link_${id}</frameId>
+        </plugin>
+      </sensor>
+    </gazebo>
+  </xacro:macro>
   <!-- ######################################################################## -->
   <!-- Main quadrotor link -->
@@ -141,4 +202,5 @@
     <xacro:quadrotor_single_propeller propid="3" id="${id}" xyz="0.00 -0.40 0.03" />
     <xacro:generic_camera  id="${id}" />
+    <xacro:sonar_sensor id="${id}" />
     <gazebo reference="base_link_${id}">
       <turnGravityOff>false</turnGravityOff>

Commit message: First Model Firefly

File: visualization/urdf/grvc_quadrotor_base.urdf.xacro (robot description, xacro)
@@ -187,5 +187,5 @@
         <origin xyz="0 0 -0.25" rpy="0 0 0" />
         <geometry>
-          <mesh filename="package://grvc_quadrotor_gazebo/model/grvc_quad.dae"/>
+          <mesh filename="package://mbzirc_gcs_view/model/firefly_scale.dae"/>
         </geometry>
       </visual>
@@ -193,12 +193,14 @@
         <origin xyz="0 0 -0.25" rpy="0 0 0" />
         <geometry>
-          <mesh filename="package://grvc_quadrotor_gazebo/model/grvc_quad_simplified.stl"/>
+          <mesh filename="package://mbzirc_gcs_view/model/firefly_scale.dae"/>
         </geometry>
       </collision>
     </link>
-    <xacro:quadrotor_single_propeller propid="0" id="${id}" xyz="0.40 0.00 0.03" />
-    <xacro:quadrotor_single_propeller propid="1" id="${id}" xyz="0.00 0.41 0.03" />
-    <xacro:quadrotor_single_propeller propid="2" id="${id}" xyz="-0.40 0.00 0.03" />
-    <xacro:quadrotor_single_propeller propid="3" id="${id}" xyz="0.00 -0.40 0.03" />
+    <xacro:quadrotor_single_propeller propid="0" id="${id}" xyz="0.40 0.23 -0.05" />
+    <xacro:quadrotor_single_propeller propid="1" id="${id}" xyz="0.00 0.46 -0.05" />
+    <xacro:quadrotor_single_propeller propid="2" id="${id}" xyz="-0.40 0.23 -0.05" />
+    <xacro:quadrotor_single_propeller propid="3" id="${id}" xyz="0.00 -0.46 -0.05" />
+    <xacro:quadrotor_single_propeller propid="4" id="${id}" xyz="-0.40 -0.23 -0.05" />
+    <xacro:quadrotor_single_propeller propid="5" id="${id}" xyz="0.40 -0.23 -0.05" />
     <xacro:generic_camera  id="${id}" />
     <xacro:sonar_sensor id="${id}" />

Commit message: New propellers for urdf

File: visualization/urdf/grvc_quadrotor_base.urdf.xacro (robot description, xacro)
@@ -27,5 +27,5 @@
     <link name="prop_${propid}_${id}">
       <inertial>
-        <mass value="0.00001" />
+        <mass value="0.0000" />
         <origin xyz="0.0 0.0 0.0" rpy="0.0 0.0 0.0" />
         <inertia ixx="0.0" ixy="0.0" ixz="0.0" iyy="0.0" iyz="0.0" izz="0.0" />
@@ -34,5 +34,5 @@
         <origin xyz="0.0 0.0 0.0" rpy="0.0 0.0 0.0" />
         <geometry>
-          <mesh filename="package://grvc_quadrotor_gazebo/model/propellers.dae"/>
+          <mesh filename="package://mbzirc_gcs_view/model/propeller_scale.dae"/>
         </geometry>
       </visual>
@@ -197,10 +197,10 @@
       </collision>
     </link>
-    <xacro:quadrotor_single_propeller propid="0" id="${id}" xyz="0.40 0.23 -0.05" />
-    <xacro:quadrotor_single_propeller propid="1" id="${id}" xyz="0.00 0.46 -0.05" />
-    <xacro:quadrotor_single_propeller propid="2" id="${id}" xyz="-0.40 0.23 -0.05" />
-    <xacro:quadrotor_single_propeller propid="3" id="${id}" xyz="0.00 -0.46 -0.05" />
-    <xacro:quadrotor_single_propeller propid="4" id="${id}" xyz="-0.40 -0.23 -0.05" />
-    <xacro:quadrotor_single_propeller propid="5" id="${id}" xyz="0.40 -0.23 -0.05" />
+    <xacro:quadrotor_single_propeller propid="0" id="${id}" xyz="0.33 0.11 -0.18" />
+    <xacro:quadrotor_single_propeller propid="1" id="${id}" xyz="-0.07 0.34 -0.18" />
+    <xacro:quadrotor_single_propeller propid="2" id="${id}" xyz="-0.47 0.11 -0.18" />
+    <xacro:quadrotor_single_propeller propid="3" id="${id}" xyz="-0.07 -0.58 -0.18" />
+    <xacro:quadrotor_single_propeller propid="4" id="${id}" xyz="-0.47 -0.35 -0.18" />
+    <xacro:quadrotor_single_propeller propid="5" id="${id}" xyz="0.33 -0.35 -0.18" />
     <xacro:generic_camera  id="${id}" />
     <xacro:sonar_sensor id="${id}" />

Commit message: New Sonar Position

File: visualization/urdf/grvc_quadrotor_base.urdf.xacro (robot description, xacro)
@@ -136,5 +136,5 @@
     </link>
     <joint name="sonar_${id}_joint" type="fixed">
-      <origin xyz="0 0.25 0.032" rpy="0 1.57 0"/>
+      <origin xyz="0 0.35 -0.065" rpy="0 1.57 0"/>
       <parent link="base_link_${id}"/>
       <child link="sonar_link_${id}"/>

Commit message: Correct integration between Gazebo&Rviz Version 1.0

File: visualization/urdf/grvc_quadrotor_base.urdf.xacro (robot description, xacro)
@@ -46,5 +46,5 @@
     <joint name="base_prop_${propid}_joint_${id}" type="fixed">
       <origin xyz="${xyz}" rpy="0.0 0.0 0.0" />
-      <parent link="base_link_${id}"/>
+      <parent link="base_link"/>
       <child link="prop_${propid}_${id}"/>
     </joint>
@@ -75,5 +75,5 @@
     <joint name="camera_${id}_joint" type="fixed">
   		<origin xyz="0.0 0.0 -0.12" rpy="0 1.4 0"/>
-    	<parent link="base_link_${id}"/>
+        <parent link="base_link"/>
     	<child link="camera_link_${id}"/>
     </joint>
@@ -137,5 +137,5 @@
     <joint name="sonar_${id}_joint" type="fixed">
       <origin xyz="0 0.35 -0.065" rpy="0 1.57 0"/>
-      <parent link="base_link_${id}"/>
+      <parent link="base_link"/>
       <child link="sonar_link_${id}"/>
     </joint>
@@ -178,5 +178,5 @@
   <!-- Main quadrotor link -->
   <xacro:macro name="quadrotor_base_macro" params="id model_name">
-    <link name="base_link_${id}">
+    <link name="base_link">
       <inertial>
         <mass value="1.487" />
@@ -205,9 +205,9 @@
     <xacro:generic_camera  id="${id}" />
     <xacro:sonar_sensor id="${id}" />
-    <gazebo reference="base_link_${id}">
+    <gazebo reference="base_link">
       <turnGravityOff>false</turnGravityOff>
     </gazebo>
     <!-- Gazebo Plugins -->
-    <xacro:quadrotor_plugins model_name="${model_name}" base_link="base_link_${id}"/>
+    <xacro:quadrotor_plugins model_name="${model_name}" base_link="base_link"/>
   </xacro:macro>
 </robot>

Commit message: Correct conection between different base_link to fixed_frame

File: visualization/urdf/grvc_quadrotor_base.urdf.xacro (robot description, xacro)
@@ -46,5 +46,5 @@
     <joint name="base_prop_${propid}_joint_${id}" type="fixed">
       <origin xyz="${xyz}" rpy="0.0 0.0 0.0" />
-      <parent link="base_link"/>
+      <parent link="base_link_${id}"/>
       <child link="prop_${propid}_${id}"/>
     </joint>
@@ -75,5 +75,5 @@
     <joint name="camera_${id}_joint" type="fixed">
   		<origin xyz="0.0 0.0 -0.12" rpy="0 1.4 0"/>
-        <parent link="base_link"/>
+        <parent link="base_link_${id}"/>
     	<child link="camera_link_${id}"/>
     </joint>
@@ -137,5 +137,5 @@
     <joint name="sonar_${id}_joint" type="fixed">
       <origin xyz="0 0.35 -0.065" rpy="0 1.57 0"/>
-      <parent link="base_link"/>
+      <parent link="base_link_${id}"/>
       <child link="sonar_link_${id}"/>
     </joint>
@@ -178,5 +178,5 @@
   <!-- Main quadrotor link -->
   <xacro:macro name="quadrotor_base_macro" params="id model_name">
-    <link name="base_link">
+    <link name="base_link_${id}">
       <inertial>
         <mass value="1.487" />
@@ -205,9 +205,9 @@
     <xacro:generic_camera  id="${id}" />
     <xacro:sonar_sensor id="${id}" />
-    <gazebo reference="base_link">
+    <gazebo reference="base_link_${id}">
       <turnGravityOff>false</turnGravityOff>
     </gazebo>
     <!-- Gazebo Plugins -->
-    <xacro:quadrotor_plugins model_name="${model_name}" base_link="base_link"/>
+    <xacro:quadrotor_plugins model_name="${model_name}" base_link="base_link_${id}"/>
   </xacro:macro>
 </robot>

Commit message: Take more than one static objects

File: visualization/urdf/grvc_quadrotor_base.urdf.xacro (robot description, xacro)
@@ -24,5 +24,5 @@
   <!-- ######################################################################## -->
   <!-- A single propeller -->
-  <xacro:macro name="quadrotor_single_propeller" params="propid id xyz">
+  <!--xacro:macro name="quadrotor_single_propeller" params="propid id xyz">
     <link name="prop_${propid}_${id}">
       <inertial>
@@ -49,5 +49,5 @@
       <child link="prop_${propid}_${id}"/>
     </joint>
-  </xacro:macro>
+  </xacro:macro-->
 <!--##############################CAMERA#######################################################-->
   <!-- Camera -->
@@ -197,10 +197,10 @@
       </collision>
     </link>
-    <xacro:quadrotor_single_propeller propid="0" id="${id}" xyz="0.33 0.11 -0.18" />
+    <!--xacro:quadrotor_single_propeller propid="0" id="${id}" xyz="0.33 0.11 -0.18" />
     <xacro:quadrotor_single_propeller propid="1" id="${id}" xyz="-0.07 0.34 -0.18" />
     <xacro:quadrotor_single_propeller propid="2" id="${id}" xyz="-0.47 0.11 -0.18" />
     <xacro:quadrotor_single_propeller propid="3" id="${id}" xyz="-0.07 -0.58 -0.18" />
     <xacro:quadrotor_single_propeller propid="4" id="${id}" xyz="-0.47 -0.35 -0.18" />
-    <xacro:quadrotor_single_propeller propid="5" id="${id}" xyz="0.33 -0.35 -0.18" />
+    <xacro:quadrotor_single_propeller propid="5" id="${id}" xyz="0.33 -0.35 -0.18" /-->
     <xacro:generic_camera  id="${id}" />
     <xacro:sonar_sensor id="${id}" />
