Commit message: Different mesh color for each UAV

File: visualization/urdf/grvc_quadrotor.urdf.xacro (robot description, xacro)
@@ -10,9 +10,9 @@
   <xacro:property name="M_PI" value="3.1415926535897931" />
   <xacro:arg name="model_name" default="grvc_gazebo"/>
+  <xacro:arg name="mesh_name" default="1"/>
   <xacro:arg name="id" default="1"/>
   <!-- Included URDF Files -->
   <xacro:include filename="$(find mbzirc_gcs_view)/urdf/grvc_quadrotor_base.urdf.xacro" />
   <!-- Instantiate quadrotor_base_macro once (has no parameters atm) -->
-  <!-- model_name must be ual_${id} for ual node to find the uav -->
-  <xacro:quadrotor_base_macro id="$(arg id)" model_name="$(arg model_name)"/>
+  <xacro:quadrotor_base_macro id="$(arg id)" model_name="$(arg model_name)" mesh_name="$(arg mesh_name)"/>
 </robot>

File: visualization/urdf/grvc_quadrotor_base.urdf.xacro (robot description, xacro)
@@ -177,5 +177,5 @@
   <!-- ########################UAV################################################ -->
   <!-- Main quadrotor link -->
-  <xacro:macro name="quadrotor_base_macro" params="id model_name">
+  <xacro:macro name="quadrotor_base_macro" params="id model_name mesh_name">
     <link name="base_link_${id}">
       <inertial>
@@ -187,5 +187,5 @@
         <origin xyz="0 0 -0.25" rpy="0 0 0" />
         <geometry>
-          <mesh filename="package://mbzirc_gcs_view/model/firefly_scale.dae"/>
+          <mesh filename="package://mbzirc_gcs_view/model/firefly_scale_${mesh_name}.dae"/>
         </geometry>
       </visual>
@@ -193,5 +193,5 @@
         <origin xyz="0 0 -0.25" rpy="0 0 0" />
         <geometry>
-          <mesh filename="package://mbzirc_gcs_view/model/firefly_scale.dae"/>
+          <mesh filename="package://mbzirc_gcs_view/model/firefly_scale_${mesh_name}.dae"/>
         </geometry>
       </collision>
