Commit message: All objects moving

File: visualization/urdf/object_big_black_base.urdf.xacro (robot description, xacro)
@@ -27,10 +27,10 @@
       </material>
     </visual>
-    <collision>
+    <!--collision>
       <origin xyz="0 0 0" rpy="0 0 0" />
       <geometry>
           <box size="2 0.2 0.2"/>
       </geometry>
-    </collision>
+    </collision-->
   </link>
     <gazebo reference="base_link_${id}">

File: visualization/urdf/object_big_blue_base.urdf.xacro (robot description, xacro)
@@ -27,10 +27,10 @@
       </material>
     </visual>
-    <collision>
+    <!--collision>
       <origin xyz="0 0 0" rpy="0 0 0" />
       <geometry>
           <box size="2 0.2 0.20"/>
       </geometry>
-    </collision>
+    </collision-->
   </link>
     <gazebo reference="base_link_${id}">

File: visualization/urdf/object_big_red_base.urdf.xacro (robot description, xacro)
@@ -27,10 +27,10 @@
       </material>
     </visual>
-    <collision>
+    <!--collision>
       <origin xyz="0 0 0" rpy="0 0 0" />
       <geometry>
           <box size="2 0.2 0.2"/>
       </geometry>
-    </collision>
+    </collision-->
   </link>
     <gazebo reference="base_link_${id}">

File: visualization/urdf/object_black_box_base.urdf.xacro (robot description, xacro)
@@ -27,10 +27,10 @@
       </material>
     </visual>
-    <collision>
+    <!--collision>
       <origin xyz="0 0 0" rpy="0 0 0" />
       <geometry>
           <box size="0.3 0.3 0.20"/>
       </geometry>
-    </collision>
+    </collision-->
   </link>
     <gazebo reference="base_link_${id}">

File: visualization/urdf/object_blue_box_base.urdf.xacro (robot description, xacro)
@@ -27,10 +27,10 @@
       </material>
     </visual>
-    <collision>
+    <!--collision>
       <origin xyz="0 0 0" rpy="0 0 0" />
       <geometry>
           <box size="0.3 0.3 0.20"/>
       </geometry>
-    </collision>
+    </collision-->
   </link>
     <gazebo reference="base_link_${id}">

File: visualization/urdf/object_blue_cylinder_base.urdf.xacro (robot description, xacro)
@@ -27,10 +27,10 @@
       </material>
     </visual>
-    <collision>
+    <!--collision>
       <origin xyz="0 0 0" rpy="0 0 0" />
       <geometry>
           <cylinder length="0.2" radius="0.15"/>
       </geometry>
-    </collision>
+    </collision-->
   </link>
     <gazebo reference="base_link_${id}">

File: visualization/urdf/object_red_box_base.urdf.xacro (robot description, xacro)
@@ -27,10 +27,10 @@
       </material>
     </visual>
-    <collision>
+    <!--collision>
       <origin xyz="0 0 0" rpy="0 0 0" />
       <geometry>
           <box size="0.3 0.3 0.20"/>
       </geometry>
-    </collision>
+    </collision-->
   </link>
     <gazebo reference="base_link_${id}">

File: visualization/urdf/object_red_cylinder_base.urdf.xacro (robot description, xacro)
@@ -27,10 +27,10 @@
       </material>
     </visual>
-    <collision>
+    <!--collision>
       <origin xyz="0 0 0" rpy="0 0 0" />
       <geometry>
           <cylinder length="0.2" radius="0.15"/>
       </geometry>
-    </collision>
+    </collision-->
   </link>
     <gazebo reference="base_link_${id}">

Commit message: New position for world model

File: visualization/urdf/object_big_black_base.urdf.xacro (robot description, xacro)
@@ -27,10 +27,10 @@
       </material>
     </visual>
-    <!--collision>
+    <collision>
       <origin xyz="0 0 0" rpy="0 0 0" />
       <geometry>
           <box size="2 0.2 0.2"/>
       </geometry>
-    </collision-->
+    </collision>
   </link>
     <gazebo reference="base_link_${id}">

File: visualization/urdf/object_big_blue_base.urdf.xacro (robot description, xacro)
@@ -27,10 +27,10 @@
       </material>
     </visual>
-    <!--collision>
+    <collision>
       <origin xyz="0 0 0" rpy="0 0 0" />
       <geometry>
           <box size="2 0.2 0.20"/>
       </geometry>
-    </collision-->
+    </collision>
   </link>
     <gazebo reference="base_link_${id}">

File: visualization/urdf/object_big_red_base.urdf.xacro (robot description, xacro)
@@ -27,10 +27,10 @@
       </material>
     </visual>
-    <!--collision>
+    <collision>
       <origin xyz="0 0 0" rpy="0 0 0" />
       <geometry>
           <box size="2 0.2 0.2"/>
       </geometry>
-    </collision-->
+    </collision>
   </link>
     <gazebo reference="base_link_${id}">

File: visualization/urdf/object_black_box_base.urdf.xacro (robot description, xacro)
@@ -27,10 +27,10 @@
       </material>
     </visual>
-    <!--collision>
+    <collision>
       <origin xyz="0 0 0" rpy="0 0 0" />
       <geometry>
           <box size="0.3 0.3 0.20"/>
       </geometry>
-    </collision-->
+    </collision>
   </link>
     <gazebo reference="base_link_${id}">

File: visualization/urdf/object_black_cylinder_base.urdf.xacro (robot description, xacro)
@@ -27,10 +27,10 @@
     </material>
   </visual>
-  <!--collision>
+  <collision>
     <origin xyz="0 0 0" rpy="0 0 0" />
     <geometry>
         <cylinder length="0.2" radius="0.15"/>
     </geometry>
-  </collision-->
+  </collision>
 </link>
   <gazebo reference="base_link_${id}">

File: visualization/urdf/object_blue_box_base.urdf.xacro (robot description, xacro)
@@ -27,10 +27,10 @@
       </material>
     </visual>
-    <!--collision>
+    <collision>
       <origin xyz="0 0 0" rpy="0 0 0" />
       <geometry>
           <box size="0.3 0.3 0.20"/>
       </geometry>
-    </collision-->
+    </collision>
   </link>
     <gazebo reference="base_link_${id}">

File: visualization/urdf/object_blue_cylinder_base.urdf.xacro (robot description, xacro)
@@ -27,10 +27,10 @@
       </material>
     </visual>
-    <!--collision>
+    <collision>
       <origin xyz="0 0 0" rpy="0 0 0" />
       <geometry>
           <cylinder length="0.2" radius="0.15"/>
       </geometry>
-    </collision-->
+    </collision>
   </link>
     <gazebo reference="base_link_${id}">

File: visualization/urdf/object_red_box_base.urdf.xacro (robot description, xacro)
@@ -27,10 +27,10 @@
       </material>
     </visual>
-    <!--collision>
+    <collision>
       <origin xyz="0 0 0" rpy="0 0 0" />
       <geometry>
           <box size="0.3 0.3 0.20"/>
       </geometry>
-    </collision-->
+    </collision>
   </link>
     <gazebo reference="base_link_${id}">

File: visualization/urdf/object_red_cylinder_base.urdf.xacro (robot description, xacro)
@@ -27,10 +27,10 @@
       </material>
     </visual>
-    <!--collision>
+    <collision>
       <origin xyz="0 0 0" rpy="0 0 0" />
       <geometry>
           <cylinder length="0.2" radius="0.15"/>
       </geometry>
-    </collision-->
+    </collision>
   </link>
     <gazebo reference="base_link_${id}">
