Commit message: URDF Drop Box in Gazebo

File: visualization/urdf/dropping_box_base.urdf.xacro (robot description, xacro)
@@ -10,32 +10,25 @@
 <xacro:include filename="$(find grvc_quadrotor_gazebo)/urdf/quadrotor_plugins.urdf.xacro" />
 <!--#####################################################################################-->
-  <!-- Main object link -->
-  <xacro:macro name="quadrotor_base_macro" params="id model_name">
-    <link name="base_link_${id}">
-      <inertial>
-        <mass value="0.5" />
-        <origin xyz="0 0 0.0" />
-        <inertia ixx="0.01152" ixy="0.0" ixz="0.0" iyy="0.01152" iyz="0.0" izz="0.0218" />
-      </inertial>
-      <visual>
-        <origin xyz="0 0 0" rpy="0 0 0" />
-        <geometry>
-            <box size="0.5 1 0.05"/>
-        </geometry>
-        <material name="gold">
-            <color rgba="0 1 1 1"/>
-        </material>
-      </visual>
-      <collision>
-        <origin xyz="0 0 0" rpy="0 0 0" />
-        <geometry>
-            <box size="0.5 1 0.05"/>
-        </geometry>
-        </collision>
-    </link>
-    <gazebo reference="base_link_${id}">
-      <material>Gazebo/Gold</material>
-      <turnGravityOff>false</turnGravityOff>
-    </gazebo>
+<!-- Main quadrotor link -->
+<xacro:macro name="quadrotor_base_macro" params="id model_name">
+  <link name="base_link_${id}">
+    <inertial>
+      <mass value="1.487" />
+      <origin xyz="0 0 0.0" />
+      <inertia ixx="0.01152" ixy="0.0" ixz="0.0" iyy="0.01152" iyz="0.0" izz="0.0218" />
+    </inertial>
+    <visual>
+      <origin xyz="0 0 -0.25" rpy="0 0 0" />
+      <geometry>
+        <mesh filename="package://mbzirc_gcs_view/model/drop_box_scale.dae"/>
+      </geometry>
+    </visual>
+    <collision>
+      <origin xyz="0 0 -0.25" rpy="0 0 0" />
+      <geometry>
+        <mesh filename="package://mbzirc_gcs_view/model/drop_box_scale.dae"/>
+      </geometry>
+    </collision>
+  </link>
     <!-- Gazebo Plugins -->
     <xacro:quadrotor_plugins model_name="${model_name}" base_link="base_link_${id}"/>

File: visualization/urdf/grvc_quadrotor_base.urdf.xacro (robot description, xacro)
@@ -175,46 +175,4 @@
     </gazebo>
   </xacro:macro>
-<!-- ###########################GRIPPER########################################### -->
-  <xacro:macro name="gripper" params="id">
-    <link name="gripper_pole_${id}">
-      <inertial>
-        <mass value="0.000" />
-        <origin xyz="0 0 0" rpy="0 0 0" />
-        <inertia ixx="0.00000000" ixy="0" ixz="0" iyy="0.00000000" iyz="0" izz="0.00000000" />
-      </inertial>
-      <visual>
-        <origin xyz="0 0 0" rpy="0 0 0" />
-        <geometry>
-          <cylinder length="0.2" radius=".01"/>
-        </geometry>
-      </visual>
-      <collision>
-        <origin xyz="0 0 0" rpy="0 0 0" />
-        <geometry>
-          <cylinder length="0.2" radius=".01"/>
-        </geometry>
-      </collision>
-    </link>
-    <link name="left_gripper_${id}">
-        <visual>
-          <origin rpy="0.0 0 0" xyz="0 0 0"/>
-          <geometry>
-            <mesh filename="package://pr2_description/meshes/gripper_v0/l_finger.dae"/>
-          </geometry>
-        </visual>
-    </link>
-    <joint name="left_gripper_joint_${id}" type="fixed">
-        <!--axis xyz="0 0 1"/>
-        <limit effort="1000.0" lower="0.0" upper="0.548" velocity="0.5"/-->
-        <origin rpy="0 0 0" xyz="0.2 0.01 0"/>
-        <parent link="gripper_pole_${id}"/>
-        <child link="left_gripper_${id}"/>
-    </joint>
-    <joint name="gripper_${id}_joint" type="fixed">
-      <origin xyz="0 0 -0.065" rpy="0 0 0"/>
-      <parent link="base_link_${id}"/>
-      <child link="gripper_pole_${id}"/>
-    </joint>
-  </xacro:macro>
   <!-- ########################UAV################################################ -->
   <!-- Main quadrotor link -->
@@ -247,5 +205,4 @@
     <xacro:generic_camera  id="${id}" />
     <xacro:sonar_sensor id="${id}" />
-    <xacro:gripper id="${id}" />
     <gazebo reference="base_link_${id}">
       <turnGravityOff>false</turnGravityOff>

Commit message: URDF Drop Box in Rviz

File: visualization/urdf/dropping_box_base.urdf.xacro (robot description, xacro)
@@ -14,10 +14,10 @@
   <link name="base_link_${id}">
     <inertial>
-      <mass value="1.487" />
+      <mass value="2" />
       <origin xyz="0 0 0.0" />
       <inertia ixx="0.01152" ixy="0.0" ixz="0.0" iyy="0.01152" iyz="0.0" izz="0.0218" />
     </inertial>
     <visual>
-      <origin xyz="0 0 -0.25" rpy="0 0 0" />
+      <origin xyz="0 0 0" rpy="0 0 0" />
       <geometry>
         <mesh filename="package://mbzirc_gcs_view/model/drop_box_scale.dae"/>
@@ -25,5 +25,5 @@
     </visual>
     <collision>
-      <origin xyz="0 0 -0.25" rpy="0 0 0" />
+      <origin xyz="0 0 0" rpy="0 0 0" />
       <geometry>
         <mesh filename="package://mbzirc_gcs_view/model/drop_box_scale.dae"/>

Commit message: New position static models (objects & box)

File: visualization/urdf/dropping_box_base.urdf.xacro (robot description, xacro)
@@ -19,5 +19,5 @@
     </inertial>
     <visual>
-      <origin xyz="0 0 0" rpy="0 0 0" />
+      <origin xyz="0 0 0" rpy="0 0 1.57" />
       <geometry>
         <mesh filename="package://mbzirc_gcs_view/model/drop_box_scale.dae"/>

File: visualization/urdf/object_big_black_base.urdf.xacro (robot description, xacro)
@@ -19,5 +19,5 @@
       </inertial>
       <visual>
-      <origin xyz="0 0 0" rpy="0 0 0" />
+      <origin xyz="0 0 0" rpy="0 0 1.57" />
       <geometry>
           <box size="2 0.2 0.2"/>
