Commit message: Change of pieces of black color by green & delete square objects

File: visualization/urdf/object_green_cylinder.urdf.xacro (robot description, xacro)
@@ -8,8 +8,8 @@
 -->
 <robot name="grvc_quadrotor" xmlns:xacro="http://ros.org/wiki/xacro">
-  <xacro:arg name="model_name" default="object_blue_cylinder_mov"/>
+  <xacro:arg name="model_name" default="object_green_cylinder_mov"/>
   <xacro:arg name="id" default="1"/>
   <!-- Included URDF Files -->
-  <xacro:include filename="$(find mbzirc_gcs_view)/urdf/object_black_box_base.urdf.xacro" />
+  <xacro:include filename="$(find mbzirc_gcs_view)/urdf/object_green_cylinder_base.urdf.xacro" />
   <!-- Instantiate quadrotor_base_macro once (has no parameters atm) -->
   <!-- model_name must be ual_${id} for ual node to find the uav -->

File: visualization/urdf/object_green_cylinder_base.urdf.xacro (robot description, xacro)
@@ -35,5 +35,5 @@
 </link>
   <gazebo reference="base_link_${id}">
-    <material>Gazebo/Black</material>
+    <material>Gazebo/Green</material>
     <turnGravityOff>false</turnGravityOff>
   </gazebo>
