Commit message: First mobile object in Arena MBZIRC

File: visualization/urdf/object_blue_cylinder_base.urdf.xacro (robot description, xacro)
@@ -10,5 +10,5 @@
 <xacro:include filename="$(find grvc_quadrotor_gazebo)/urdf/quadrotor_plugins.urdf.xacro" />
 <!--#####################################################################################-->
-  <!-- Main quadrotor link -->
+  <!-- Main object link -->
   <xacro:macro name="quadrotor_base_macro" params="id model_name">
     <link name="base_link_${id}">
@@ -21,5 +21,5 @@
       <origin xyz="0 0 0" rpy="0 0 0" />
       <geometry>
-          <box size="0.3 0.3 0.20"/>
+          <cylinder length="0.2" radius="0.15"/>
       </geometry>
       <material name="blue">
@@ -30,9 +30,10 @@
       <origin xyz="0 0 0" rpy="0 0 0" />
       <geometry>
-          <box size="0.3 0.3 0.20"/>
+          <cylinder length="0.2" radius="0.15"/>
       </geometry>
     </collision>
   </link>
     <gazebo reference="base_link_${id}">
+      <material>Gazebo/Blue</material>
       <turnGravityOff>false</turnGravityOff>
     </gazebo>

Commit message: Modify size static objects

File: visualization/urdf/object_blue_cylinder_base.urdf.xacro (robot description, xacro)
@@ -21,5 +21,5 @@
       <origin xyz="0 0 0" rpy="0 0 0" />
       <geometry>
-          <cylinder length="0.2" radius="0.15"/>
+          <cylinder length="0.2" radius="0.10"/>
       </geometry>
       <material name="blue">
@@ -30,5 +30,5 @@
       <origin xyz="0 0 0" rpy="0 0 0" />
       <geometry>
-          <cylinder length="0.2" radius="0.15"/>
+          <cylinder length="0.2" radius="0.10"/>
       </geometry>
     </collision>

File: visualization/urdf/object_green_cylinder_base.urdf.xacro (robot description, xacro)
@@ -21,5 +21,5 @@
     <origin xyz="0 0 0" rpy="0 0 0" />
     <geometry>
-        <cylinder length="0.2" radius="0.15"/>
+        <cylinder length="0.2" radius="0.1"/>
     </geometry>
     <material name="black">
@@ -30,5 +30,5 @@
     <origin xyz="0 0 0" rpy="0 0 0" />
     <geometry>
-        <cylinder length="0.2" radius="0.15"/>
+        <cylinder length="0.2" radius="0.1"/>
     </geometry>
   </collision>

File: visualization/urdf/object_red_cylinder_base.urdf.xacro (robot description, xacro)
@@ -21,5 +21,5 @@
       <origin xyz="0 0 0" rpy="0 0 0" />
       <geometry>
-          <cylinder length="0.2" radius="0.15"/>
+          <cylinder length="0.2" radius="0.10"/>
       </geometry>
       <material name="red">
@@ -30,5 +30,5 @@
       <origin xyz="0 0 0" rpy="0 0 0" />
       <geometry>
-          <cylinder length="0.2" radius="0.15"/>
+          <cylinder length="0.2" radius="0.10"/>
       </geometry>
     </collision>

Commit message: Delete old dependencies objects_base_xacro wiht quadrotor plugins

File: visualization/urdf/object_blue_cylinder_base.urdf.xacro (robot description, xacro)
@@ -8,6 +8,4 @@
 -->
 <robot xmlns:xacro="http://ros.org/wiki/xacro">
-<xacro:include filename="$(find grvc_quadrotor_gazebo)/urdf/quadrotor_plugins.urdf.xacro" />
-<!--#####################################################################################-->
   <!-- Main object link -->
   <xacro:macro name="quadrotor_base_macro" params="id model_name">
@@ -38,6 +36,4 @@
       <turnGravityOff>false</turnGravityOff>
     </gazebo>
-    <!-- Gazebo Plugins -->
-    <xacro:quadrotor_plugins model_name="${model_name}" base_link="base_link_${id}"/>
   </xacro:macro>
 </robot>

File: visualization/urdf/object_green_cylinder_base.urdf.xacro (robot description, xacro)
@@ -8,6 +8,4 @@
 -->
 <robot xmlns:xacro="http://ros.org/wiki/xacro">
-<xacro:include filename="$(find grvc_quadrotor_gazebo)/urdf/quadrotor_plugins.urdf.xacro" />
-<!--#####################################################################################-->
 <!-- Main object link -->
 <xacro:macro name="quadrotor_base_macro" params="id model_name">
@@ -23,6 +21,6 @@
         <cylinder length="0.2" radius="0.1"/>
     </geometry>
-    <material name="black">
-        <color rgba="0 0 0 1"/>
+    <material name="green">
+        <color rgba="0 0.8 0 1"/>
     </material>
   </visual>
@@ -38,6 +36,4 @@
     <turnGravityOff>false</turnGravityOff>
   </gazebo>
-  <!-- Gazebo Plugins -->
-  <xacro:quadrotor_plugins model_name="${model_name}" base_link="base_link_${id}"/>
 </xacro:macro>
 </robot>

File: visualization/urdf/object_red_cylinder_base.urdf.xacro (robot description, xacro)
@@ -8,6 +8,4 @@
 -->
 <robot xmlns:xacro="http://ros.org/wiki/xacro">
-<xacro:include filename="$(find grvc_quadrotor_gazebo)/urdf/quadrotor_plugins.urdf.xacro" />
-<!--#####################################################################################-->
   <!-- Main object link -->
   <xacro:macro name="quadrotor_base_macro" params="id model_name">
@@ -38,6 +36,4 @@
       <turnGravityOff>false</turnGravityOff>
     </gazebo>
-    <!-- Gazebo Plugins -->
-    <xacro:quadrotor_plugins model_name="${model_name}" base_link="base_link_${id}"/>
   </xacro:macro>
 </robot>
