Commit message: Delete more old dependencies in static_objects

File: visualization/urdf/object_blue_cylinder.urdf.xacro (robot description, xacro)
@@ -7,11 +7,10 @@
 THE SOFTWARE IS PROVIDED "AS IS", WITHOUT WARRANTY OF ANY KIND, EXPRESS OR IMPLIED, INCLUDING BUT NOT LIMITED TO THE WARRANTIES OF MERCHANTABILITY, FITNESS FOR A PARTICULAR PURPOSE AND NONINFRINGEMENT. IN NO EVENT SHALL THE AUTHORS OR COPYRIGHT HOLDERS BE LIABLE FOR ANY CLAIM, DAMAGES OR OTHER LIABILITY, WHETHER IN AN ACTION OF CONTRACT, TORT OR OTHERWISE, ARISING FROM, OUT OF OR IN CONNECTION WITH THE SOFTWARE OR THE USE OR OTHER DEALINGS IN THE SOFTWARE.
 -->
-<robot name="grvc_quadrotor" xmlns:xacro="http://ros.org/wiki/xacro">
+<robot name="blue_cylinder" xmlns:xacro="http://ros.org/wiki/xacro">
   <xacro:arg name="model_name" default="object_blue_cylinder_mov"/>
   <xacro:arg name="id" default="1"/>
   <!-- Included URDF Files -->
   <xacro:include filename="$(find mbzirc_gcs_view)/urdf/object_blue_cylinder_base.urdf.xacro" />
-  <!-- Instantiate quadrotor_base_macro once (has no parameters atm) -->
   <!-- model_name must be ual_${id} for ual node to find the uav -->
-  <xacro:quadrotor_base_macro id="$(arg id)" model_name="$(arg model_name)"/>
+  <xacro:blue_cylinder id="$(arg id)" model_name="$(arg model_name)"/>
 </robot>

File: visualization/urdf/object_blue_cylinder_base.urdf.xacro (robot description, xacro)
@@ -9,5 +9,5 @@
 <robot xmlns:xacro="http://ros.org/wiki/xacro">
   <!-- Main object link -->
-  <xacro:macro name="quadrotor_base_macro" params="id model_name">
+  <xacro:macro name="blue_cylinder" params="id model_name">
     <link name="base_link_${id}">
       <inertial>

File: visualization/urdf/object_green_cylinder.urdf.xacro (robot description, xacro)
@@ -7,11 +7,10 @@
 THE SOFTWARE IS PROVIDED "AS IS", WITHOUT WARRANTY OF ANY KIND, EXPRESS OR IMPLIED, INCLUDING BUT NOT LIMITED TO THE WARRANTIES OF MERCHANTABILITY, FITNESS FOR A PARTICULAR PURPOSE AND NONINFRINGEMENT. IN NO EVENT SHALL THE AUTHORS OR COPYRIGHT HOLDERS BE LIABLE FOR ANY CLAIM, DAMAGES OR OTHER LIABILITY, WHETHER IN AN ACTION OF CONTRACT, TORT OR OTHERWISE, ARISING FROM, OUT OF OR IN CONNECTION WITH THE SOFTWARE OR THE USE OR OTHER DEALINGS IN THE SOFTWARE.
 -->
-<robot name="grvc_quadrotor" xmlns:xacro="http://ros.org/wiki/xacro">
+<robot name="green_cylinder" xmlns:xacro="http://ros.org/wiki/xacro">
   <xacro:arg name="model_name" default="object_green_cylinder_mov"/>
   <xacro:arg name="id" default="1"/>
   <!-- Included URDF Files -->
   <xacro:include filename="$(find mbzirc_gcs_view)/urdf/object_green_cylinder_base.urdf.xacro" />
-  <!-- Instantiate quadrotor_base_macro once (has no parameters atm) -->
   <!-- model_name must be ual_${id} for ual node to find the uav -->
-  <xacro:quadrotor_base_macro id="$(arg id)" model_name="$(arg model_name)"/>
+  <xacro:green_cylinder id="$(arg id)" model_name="$(arg model_name)"/>
 </robot>

File: visualization/urdf/object_green_cylinder_base.urdf.xacro (robot description, xacro)
@@ -9,5 +9,5 @@
 <robot xmlns:xacro="http://ros.org/wiki/xacro">
 <!-- Main object link -->
-<xacro:macro name="quadrotor_base_macro" params="id model_name">
+<xacro:macro name="green_cylinder" params="id model_name">
   <link name="base_link_${id}">
     <inertial>

File: visualization/urdf/object_red_cylinder.urdf.xacro (robot description, xacro)
@@ -7,11 +7,10 @@
 THE SOFTWARE IS PROVIDED "AS IS", WITHOUT WARRANTY OF ANY KIND, EXPRESS OR IMPLIED, INCLUDING BUT NOT LIMITED TO THE WARRANTIES OF MERCHANTABILITY, FITNESS FOR A PARTICULAR PURPOSE AND NONINFRINGEMENT. IN NO EVENT SHALL THE AUTHORS OR COPYRIGHT HOLDERS BE LIABLE FOR ANY CLAIM, DAMAGES OR OTHER LIABILITY, WHETHER IN AN ACTION OF CONTRACT, TORT OR OTHERWISE, ARISING FROM, OUT OF OR IN CONNECTION WITH THE SOFTWARE OR THE USE OR OTHER DEALINGS IN THE SOFTWARE.
 -->
-<robot name="grvc_quadrotor" xmlns:xacro="http://ros.org/wiki/xacro">
+<robot name="red_cylinder" xmlns:xacro="http://ros.org/wiki/xacro">
   <xacro:arg name="model_name" default="object_red_cylinder_mov"/>
   <xacro:arg name="id" default="1"/>
   <!-- Included URDF Files -->
   <xacro:include filename="$(find mbzirc_gcs_view)/urdf/object_red_cylinder_base.urdf.xacro" />
-  <!-- Instantiate quadrotor_base_macro once (has no parameters atm) -->
   <!-- model_name must be ual_${id} for ual node to find the uav -->
-  <xacro:quadrotor_base_macro id="$(arg id)" model_name="$(arg model_name)"/>
+  <xacro:red_cylinder id="$(arg id)" model_name="$(arg model_name)"/>
 </robot>

File: visualization/urdf/object_red_cylinder_base.urdf.xacro (robot description, xacro)
@@ -9,5 +9,5 @@
 <robot xmlns:xacro="http://ros.org/wiki/xacro">
   <!-- Main object link -->
-  <xacro:macro name="quadrotor_base_macro" params="id model_name">
+  <xacro:macro name="red_cylinder" params="id model_name">
     <link name="base_link_${id}">
       <inertial>

Commit message: Added urdf yellow objects

File: visualization/urdf/object_blue_cylinder.urdf.xacro (robot description, xacro)
@@ -1,10 +1,3 @@
 <?xml version="1.0"?>
-<!--
-The MIT License (MIT)
-Copyright (c) 2016 GRVC University of Seville
-Permission is hereby granted, free of charge, to any person obtaining a copy of this software and associated documentation files (the "Software"), to deal in the Software without restriction, including without limitation the rights to use, copy, modify, merge, publish, distribute, sublicense, and/or sell copies of the Software, and to permit persons to whom the Software is furnished to do so, subject to the following conditions:
-The above copyright notice and this permission notice shall be included in all copies or substantial portions of the Software.
-THE SOFTWARE IS PROVIDED "AS IS", WITHOUT WARRANTY OF ANY KIND, EXPRESS OR IMPLIED, INCLUDING BUT NOT LIMITED TO THE WARRANTIES OF MERCHANTABILITY, FITNESS FOR A PARTICULAR PURPOSE AND NONINFRINGEMENT. IN NO EVENT SHALL THE AUTHORS OR COPYRIGHT HOLDERS BE LIABLE FOR ANY CLAIM, DAMAGES OR OTHER LIABILITY, WHETHER IN AN ACTION OF CONTRACT, TORT OR OTHERWISE, ARISING FROM, OUT OF OR IN CONNECTION WITH THE SOFTWARE OR THE USE OR OTHER DEALINGS IN THE SOFTWARE.
--->
 <robot name="blue_cylinder" xmlns:xacro="http://ros.org/wiki/xacro">
   <xacro:arg name="model_name" default="object_blue_cylinder_mov"/>

File: visualization/urdf/object_blue_cylinder_base.urdf.xacro (robot description, xacro)
@@ -1,10 +1,3 @@
 <?xml version="1.0"?>
-<!--
-The MIT License (MIT)
-Copyright (c) 2016 GRVC University of Seville
-Permission is hereby granted, free of charge, to any person obtaining a copy of this software and associated documentation files (the "Software"), to deal in the Software without restriction, including without limitation the rights to use, copy, modify, merge, publish, distribute, sublicense, and/or sell copies of the Software, and to permit persons to whom the Software is furnished to do so, subject to the following conditions:
-The above copyright notice and this permission notice shall be included in all copies or substantial portions of the Software.
-THE SOFTWARE IS PROVIDED "AS IS", WITHOUT WARRANTY OF ANY KIND, EXPRESS OR IMPLIED, INCLUDING BUT NOT LIMITED TO THE WARRANTIES OF MERCHANTABILITY, FITNESS FOR A PARTICULAR PURPOSE AND NONINFRINGEMENT. IN NO EVENT SHALL THE AUTHORS OR COPYRIGHT HOLDERS BE LIABLE FOR ANY CLAIM, DAMAGES OR OTHER LIABILITY, WHETHER IN AN ACTION OF CONTRACT, TORT OR OTHERWISE, ARISING FROM, OUT OF OR IN CONNECTION WITH THE SOFTWARE OR THE USE OR OTHER DEALINGS IN THE SOFTWARE.
--->
 <robot xmlns:xacro="http://ros.org/wiki/xacro">
   <!-- Main object link -->

File: visualization/urdf/object_green_cylinder.urdf.xacro (robot description, xacro)
@@ -1,16 +1,8 @@
 <?xml version="1.0"?>
-<!--
-The MIT License (MIT)
-Copyright (c) 2016 GRVC University of Seville
-Permission is hereby granted, free of charge, to any person obtaining a copy of this software and associated documentation files (the "Software"), to deal in the Software without restriction, including without limitation the rights to use, copy, modify, merge, publish, distribute, sublicense, and/or sell copies of the Software, and to permit persons to whom the Software is furnished to do so, subject to the following conditions:
-The above copyright notice and this permission notice shall be included in all copies or substantial portions of the Software.
-THE SOFTWARE IS PROVIDED "AS IS", WITHOUT WARRANTY OF ANY KIND, EXPRESS OR IMPLIED, INCLUDING BUT NOT LIMITED TO THE WARRANTIES OF MERCHANTABILITY, FITNESS FOR A PARTICULAR PURPOSE AND NONINFRINGEMENT. IN NO EVENT SHALL THE AUTHORS OR COPYRIGHT HOLDERS BE LIABLE FOR ANY CLAIM, DAMAGES OR OTHER LIABILITY, WHETHER IN AN ACTION OF CONTRACT, TORT OR OTHERWISE, ARISING FROM, OUT OF OR IN CONNECTION WITH THE SOFTWARE OR THE USE OR OTHER DEALINGS IN THE SOFTWARE.
--->
 <robot name="green_cylinder" xmlns:xacro="http://ros.org/wiki/xacro">
-  <xacro:arg name="model_name" default="object_green_cylinder_mov"/>
   <xacro:arg name="id" default="1"/>
   <!-- Included URDF Files -->
   <xacro:include filename="$(find mbzirc_gcs_view)/urdf/object_green_cylinder_base.urdf.xacro" />
   <!-- model_name must be ual_${id} for ual node to find the uav -->
-  <xacro:green_cylinder id="$(arg id)" model_name="$(arg model_name)"/>
+  <xacro:green_cylinder id="$(arg id)"/>
 </robot>

File: visualization/urdf/object_green_cylinder_base.urdf.xacro (robot description, xacro)
@@ -1,13 +1,6 @@
 <?xml version="1.0"?>
-<!--
-The MIT License (MIT)
-Copyright (c) 2016 GRVC University of Seville
-Permission is hereby granted, free of charge, to any person obtaining a copy of this software and associated documentation files (the "Software"), to deal in the Software without restriction, including without limitation the rights to use, copy, modify, merge, publish, distribute, sublicense, and/or sell copies of the Software, and to permit persons to whom the Software is furnished to do so, subject to the following conditions:
-The above copyright notice and this permission notice shall be included in all copies or substantial portions of the Software.
-THE SOFTWARE IS PROVIDED "AS IS", WITHOUT WARRANTY OF ANY KIND, EXPRESS OR IMPLIED, INCLUDING BUT NOT LIMITED TO THE WARRANTIES OF MERCHANTABILITY, FITNESS FOR A PARTICULAR PURPOSE AND NONINFRINGEMENT. IN NO EVENT SHALL THE AUTHORS OR COPYRIGHT HOLDERS BE LIABLE FOR ANY CLAIM, DAMAGES OR OTHER LIABILITY, WHETHER IN AN ACTION OF CONTRACT, TORT OR OTHERWISE, ARISING FROM, OUT OF OR IN CONNECTION WITH THE SOFTWARE OR THE USE OR OTHER DEALINGS IN THE SOFTWARE.
--->
 <robot xmlns:xacro="http://ros.org/wiki/xacro">
 <!-- Main object link -->
-<xacro:macro name="green_cylinder" params="id model_name">
+<xacro:macro name="green_cylinder" params="id">
   <link name="base_link_${id}">
     <inertial>

File: visualization/urdf/object_yellow_cylinder.urdf.xacro (robot description, xacro)
@@ -1,8 +1,8 @@
 <?xml version="1.0"?>
-<robot name="red_cylinder" xmlns:xacro="http://ros.org/wiki/xacro">
-  <xacro:arg name="model_name" default="object_red_cylinder_mov"/>
+<robot name="yellow_cylinder" xmlns:xacro="http://ros.org/wiki/xacro">
+  <xacro:arg name="model_name" default="object_yellow_cylinder_mov"/>
   <xacro:arg name="id" default="1"/>
   <!-- Included URDF Files -->
-  <xacro:include filename="$(find mbzirc_gcs_view)/urdf/object_red_cylinder_base.urdf.xacro" />
+  <xacro:include filename="$(find mbzirc_gcs_view)/urdf/object_yellow_cylinder_base.urdf.xacro" />
   <!-- model_name must be ual_${id} for ual node to find the uav -->
   <xacro:red_cylinder id="$(arg id)" model_name="$(arg model_name)"/>

File: visualization/urdf/object_yellow_cylinder_base.urdf.xacro (robot description, xacro)
@@ -2,5 +2,5 @@
 <robot xmlns:xacro="http://ros.org/wiki/xacro">
   <!-- Main object link -->
-  <xacro:macro name="red_cylinder" params="id model_name">
+  <xacro:macro name="yellow_cylinder" params="id">
     <link name="base_link_${id}">
       <inertial>
@@ -14,6 +14,6 @@
           <cylinder length="0.2" radius="0.10"/>
       </geometry>
-      <material name="red">
-          <color rgba="0.8 0 0 1"/>
+      <material name="yellow">
+          <color rgba="0.8 0.6 0 1"/>
       </material>
     </visual>
@@ -26,5 +26,5 @@
   </link>
     <gazebo reference="base_link_${id}">
-      <material>Gazebo/Red</material>
+      <material>Gazebo/Yellow</material>
       <turnGravityOff>false</turnGravityOff>
     </gazebo>
