Commit message: Yellow static objects comments in simulation.launch

File: visualization/urdf/object_yellow_cylinder.urdf.xacro (robot description, xacro)
@@ -6,4 +6,4 @@
   <xacro:include filename="$(find mbzirc_gcs_view)/urdf/object_yellow_cylinder_base.urdf.xacro" />
   <!-- model_name must be ual_${id} for ual node to find the uav -->
-  <xacro:red_cylinder id="$(arg id)" model_name="$(arg model_name)"/>
+  <xacro:yellow_cylinder id="$(arg id)" model_name="$(arg model_name)"/>
 </robot>

File: visualization/urdf/object_yellow_cylinder_base.urdf.xacro (robot description, xacro)
@@ -2,5 +2,5 @@
 <robot xmlns:xacro="http://ros.org/wiki/xacro">
   <!-- Main object link -->
-  <xacro:macro name="yellow_cylinder" params="id">
+  <xacro:macro name="yellow_cylinder" params="id model_name">
     <link name="base_link_${id}">
       <inertial>
