Commit message: New color for big static objects

File: visualization/urdf/object_big.urdf.xacro (robot description, xacro)
@@ -11,5 +11,5 @@
   <xacro:arg name="id" default="1"/>
   <!-- Included URDF Files -->
-  <xacro:include filename="$(find mbzirc_gcs_view)/urdf/object_big_blue_base.urdf.xacro" />
+  <xacro:include filename="$(find mbzirc_gcs_view)/urdf/object_big_base.urdf.xacro" />
   <!-- Instantiate quadrotor_base_macro once (has no parameters atm) -->
   <!-- model_name must be ual_${id} for ual node to find the uav -->

File: visualization/urdf/object_big_base.urdf.xacro (robot description, xacro)
@@ -35,5 +35,5 @@
   </link>
     <gazebo reference="base_link_${id}">
-      <material>Gazebo/Black</material>
+      <material>Gazebo/Orange</material>
       <turnGravityOff>false</turnGravityOff>
     </gazebo>
