Commit message: Spawn urdf big object in Gazebo

File: visualization/urdf/dropping_box.urdf.xacro (robot description, xacro)
@@ -7,34 +7,11 @@
 THE SOFTWARE IS PROVIDED "AS IS", WITHOUT WARRANTY OF ANY KIND, EXPRESS OR IMPLIED, INCLUDING BUT NOT LIMITED TO THE WARRANTIES OF MERCHANTABILITY, FITNESS FOR A PARTICULAR PURPOSE AND NONINFRINGEMENT. IN NO EVENT SHALL THE AUTHORS OR COPYRIGHT HOLDERS BE LIABLE FOR ANY CLAIM, DAMAGES OR OTHER LIABILITY, WHETHER IN AN ACTION OF CONTRACT, TORT OR OTHERWISE, ARISING FROM, OUT OF OR IN CONNECTION WITH THE SOFTWARE OR THE USE OR OTHER DEALINGS IN THE SOFTWARE.
 -->
-<robot xmlns:xacro="http://ros.org/wiki/xacro">
-<!--#####################################################################################-->
-  <!-- Main object link -->
-  <xacro:macro name="quadrotor_base_macro" params="id model_name">
-    <link name="base_link_${id}">
-      <inertial>
-        <mass value="0.5" />
-        <origin xyz="0 0 0.0" />
-        <inertia ixx="0.01152" ixy="0.0" ixz="0.0" iyy="0.01152" iyz="0.0" izz="0.0218" />
-      </inertial>
-      <visual>
-      <origin xyz="0 0 0" rpy="0 0 0" />
-      <geometry>
-          <box size="2 0.2 0.20"/>
-      </geometry>
-      <material name="blue">
-          <color rgba="0 0 .8 0"/>
-      </material>
-    </visual>
-    <collision>
-      <origin xyz="0 0 0" rpy="0 0 0" />
-      <geometry>
-          <box size="2 0.2 0.20"/>
-      </geometry>
-    </collision>
-  </link>
-    <gazebo reference="base_link_${id}">
-      <material>Gazebo/Blue</material>
-      <turnGravityOff>false</turnGravityOff>
-    </gazebo>
-  </xacro:macro>
+<robot name="grvc_quadrotor" xmlns:xacro="http://ros.org/wiki/xacro">
+  <xacro:arg name="model_name" default="object_blue_box_mov"/>
+  <xacro:arg name="id" default="1"/>
+  <!-- Included URDF Files -->
+  <xacro:include filename="$(find mbzirc_gcs_view)/urdf/object_blue_box_base.urdf.xacro" />
+  <!-- Instantiate quadrotor_base_macro once (has no parameters atm) -->
+  <!-- model_name must be ual_${id} for ual node to find the uav -->
+  <xacro:quadrotor_base_macro id="$(arg id)" model_name="$(arg model_name)"/>
 </robot>

File: visualization/urdf/dropping_box_base.urdf.xacro (robot description, xacro)
@@ -8,4 +8,5 @@
 -->
 <robot xmlns:xacro="http://ros.org/wiki/xacro">
+<xacro:include filename="$(find grvc_quadrotor_gazebo)/urdf/quadrotor_plugins.urdf.xacro" />
 <!--#####################################################################################-->
   <!-- Main object link -->
@@ -20,8 +21,8 @@
       <origin xyz="0 0 0" rpy="0 0 0" />
       <geometry>
-          <box size="2 0.2 0.20"/>
+          <box size="0.3 0.3 0.20"/>
       </geometry>
       <material name="blue">
-          <color rgba="0 0 .8 0"/>
+          <color rgba="0 0 .8 1"/>
       </material>
     </visual>
@@ -29,5 +30,5 @@
       <origin xyz="0 0 0" rpy="0 0 0" />
       <geometry>
-          <box size="2 0.2 0.20"/>
+          <box size="0.3 0.3 0.20"/>
       </geometry>
     </collision>
@@ -37,4 +38,6 @@
       <turnGravityOff>false</turnGravityOff>
     </gazebo>
+    <!-- Gazebo Plugins -->
+    <xacro:quadrotor_plugins model_name="${model_name}" base_link="base_link_${id}"/>
   </xacro:macro>
 </robot>

File: visualization/urdf/object_big_black.urdf.xacro (robot description, xacro)
@@ -7,34 +7,11 @@
 THE SOFTWARE IS PROVIDED "AS IS", WITHOUT WARRANTY OF ANY KIND, EXPRESS OR IMPLIED, INCLUDING BUT NOT LIMITED TO THE WARRANTIES OF MERCHANTABILITY, FITNESS FOR A PARTICULAR PURPOSE AND NONINFRINGEMENT. IN NO EVENT SHALL THE AUTHORS OR COPYRIGHT HOLDERS BE LIABLE FOR ANY CLAIM, DAMAGES OR OTHER LIABILITY, WHETHER IN AN ACTION OF CONTRACT, TORT OR OTHERWISE, ARISING FROM, OUT OF OR IN CONNECTION WITH THE SOFTWARE OR THE USE OR OTHER DEALINGS IN THE SOFTWARE.
 -->
-<robot xmlns:xacro="http://ros.org/wiki/xacro">
-<!--#####################################################################################-->
-  <!-- Main object link -->
-  <xacro:macro name="quadrotor_base_macro" params="id model_name">
-    <link name="base_link_${id}">
-      <inertial>
-        <mass value="0.5" />
-        <origin xyz="0 0 0.0" />
-        <inertia ixx="0.01152" ixy="0.0" ixz="0.0" iyy="0.01152" iyz="0.0" izz="0.0218" />
-      </inertial>
-      <visual>
-      <origin xyz="0 0 0" rpy="0 0 0" />
-      <geometry>
-          <box size="2 0.2 0.20"/>
-      </geometry>
-      <material name="blue">
-          <color rgba="0 0 .8 0"/>
-      </material>
-    </visual>
-    <collision>
-      <origin xyz="0 0 0" rpy="0 0 0" />
-      <geometry>
-          <box size="2 0.2 0.20"/>
-      </geometry>
-    </collision>
-  </link>
-    <gazebo reference="base_link_${id}">
-      <material>Gazebo/Blue</material>
-      <turnGravityOff>false</turnGravityOff>
-    </gazebo>
-  </xacro:macro>
+<robot name="grvc_quadrotor" xmlns:xacro="http://ros.org/wiki/xacro">
+  <xacro:arg name="model_name" default="object_blue_cylinder_mov"/>
+  <xacro:arg name="id" default="1"/>
+  <!-- Included URDF Files -->
+  <xacro:include filename="$(find mbzirc_gcs_view)/urdf/object_big_black_base.urdf.xacro" />
+  <!-- Instantiate quadrotor_base_macro once (has no parameters atm) -->
+  <!-- model_name must be ual_${id} for ual node to find the uav -->
+  <xacro:quadrotor_base_macro id="$(arg id)" model_name="$(arg model_name)"/>
 </robot>

File: visualization/urdf/object_big_blue.urdf.xacro (robot description, xacro)
@@ -7,34 +7,11 @@
 THE SOFTWARE IS PROVIDED "AS IS", WITHOUT WARRANTY OF ANY KIND, EXPRESS OR IMPLIED, INCLUDING BUT NOT LIMITED TO THE WARRANTIES OF MERCHANTABILITY, FITNESS FOR A PARTICULAR PURPOSE AND NONINFRINGEMENT. IN NO EVENT SHALL THE AUTHORS OR COPYRIGHT HOLDERS BE LIABLE FOR ANY CLAIM, DAMAGES OR OTHER LIABILITY, WHETHER IN AN ACTION OF CONTRACT, TORT OR OTHERWISE, ARISING FROM, OUT OF OR IN CONNECTION WITH THE SOFTWARE OR THE USE OR OTHER DEALINGS IN THE SOFTWARE.
 -->
-<robot xmlns:xacro="http://ros.org/wiki/xacro">
-<!--#####################################################################################-->
-  <!-- Main object link -->
-  <xacro:macro name="quadrotor_base_macro" params="id model_name">
-    <link name="base_link_${id}">
-      <inertial>
-        <mass value="0.5" />
-        <origin xyz="0 0 0.0" />
-        <inertia ixx="0.01152" ixy="0.0" ixz="0.0" iyy="0.01152" iyz="0.0" izz="0.0218" />
-      </inertial>
-      <visual>
-      <origin xyz="0 0 0" rpy="0 0 0" />
-      <geometry>
-          <box size="2 0.2 0.20"/>
-      </geometry>
-      <material name="blue">
-          <color rgba="0 0 .8 0"/>
-      </material>
-    </visual>
-    <collision>
-      <origin xyz="0 0 0" rpy="0 0 0" />
-      <geometry>
-          <box size="2 0.2 0.20"/>
-      </geometry>
-    </collision>
-  </link>
-    <gazebo reference="base_link_${id}">
-      <material>Gazebo/Blue</material>
-      <turnGravityOff>false</turnGravityOff>
-    </gazebo>
-  </xacro:macro>
+<robot name="grvc_quadrotor" xmlns:xacro="http://ros.org/wiki/xacro">
+  <xacro:arg name="model_name" default="object_blue_cylinder_mov"/>
+  <xacro:arg name="id" default="1"/>
+  <!-- Included URDF Files -->
+  <xacro:include filename="$(find mbzirc_gcs_view)/urdf/object_big_blue_base.urdf.xacro" />
+  <!-- Instantiate quadrotor_base_macro once (has no parameters atm) -->
+  <!-- model_name must be ual_${id} for ual node to find the uav -->
+  <xacro:quadrotor_base_macro id="$(arg id)" model_name="$(arg model_name)"/>
 </robot>

File: visualization/urdf/object_big_red.urdf.xacro (robot description, xacro)
@@ -7,34 +7,11 @@
 THE SOFTWARE IS PROVIDED "AS IS", WITHOUT WARRANTY OF ANY KIND, EXPRESS OR IMPLIED, INCLUDING BUT NOT LIMITED TO THE WARRANTIES OF MERCHANTABILITY, FITNESS FOR A PARTICULAR PURPOSE AND NONINFRINGEMENT. IN NO EVENT SHALL THE AUTHORS OR COPYRIGHT HOLDERS BE LIABLE FOR ANY CLAIM, DAMAGES OR OTHER LIABILITY, WHETHER IN AN ACTION OF CONTRACT, TORT OR OTHERWISE, ARISING FROM, OUT OF OR IN CONNECTION WITH THE SOFTWARE OR THE USE OR OTHER DEALINGS IN THE SOFTWARE.
 -->
-<robot xmlns:xacro="http://ros.org/wiki/xacro">
-<!--#####################################################################################-->
-  <!-- Main object link -->
-  <xacro:macro name="quadrotor_base_macro" params="id model_name">
-    <link name="base_link_${id}">
-      <inertial>
-        <mass value="0.5" />
-        <origin xyz="0 0 0.0" />
-        <inertia ixx="0.01152" ixy="0.0" ixz="0.0" iyy="0.01152" iyz="0.0" izz="0.0218" />
-      </inertial>
-      <visual>
-      <origin xyz="0 0 0" rpy="0 0 0" />
-      <geometry>
-          <box size="2 0.2 0.20"/>
-      </geometry>
-      <material name="blue">
-          <color rgba="0 0 .8 0"/>
-      </material>
-    </visual>
-    <collision>
-      <origin xyz="0 0 0" rpy="0 0 0" />
-      <geometry>
-          <box size="2 0.2 0.20"/>
-      </geometry>
-    </collision>
-  </link>
-    <gazebo reference="base_link_${id}">
-      <material>Gazebo/Blue</material>
-      <turnGravityOff>false</turnGravityOff>
-    </gazebo>
-  </xacro:macro>
+<robot name="grvc_quadrotor" xmlns:xacro="http://ros.org/wiki/xacro">
+  <xacro:arg name="model_name" default="object_blue_cylinder_mov"/>
+  <xacro:arg name="id" default="1"/>
+  <!-- Included URDF Files -->
+  <xacro:include filename="$(find mbzirc_gcs_view)/urdf/object_big_red_base.urdf.xacro" />
+  <!-- Instantiate quadrotor_base_macro once (has no parameters atm) -->
+  <!-- model_name must be ual_${id} for ual node to find the uav -->
+  <xacro:quadrotor_base_macro id="$(arg id)" model_name="$(arg model_name)"/>
 </robot>

File: visualization/urdf/object_black_cylinder_base.urdf.xacro (robot description, xacro)
@@ -14,5 +14,5 @@
   <link name="base_link_${id}">
     <inertial>
-      <mass value="0.5" />
+      <mass value="0.1" />
       <origin xyz="0 0 0.0" />
       <inertia ixx="0.01152" ixy="0.0" ixz="0.0" iyy="0.01152" iyz="0.0" izz="0.0218" />
@@ -27,10 +27,10 @@
     </material>
   </visual>
-  <collision>
+  <!--collision>
     <origin xyz="0 0 0" rpy="0 0 0" />
     <geometry>
         <cylinder length="0.2" radius="0.15"/>
     </geometry>
-  </collision>
+  </collision-->
 </link>
   <gazebo reference="base_link_${id}">

Commit message: Pick up static object

File: visualization/urdf/dropping_box.urdf.xacro (robot description, xacro)
@@ -11,5 +11,5 @@
   <xacro:arg name="id" default="1"/>
   <!-- Included URDF Files -->
-  <xacro:include filename="$(find mbzirc_gcs_view)/urdf/object_blue_box_base.urdf.xacro" />
+  <xacro:include filename="$(find mbzirc_gcs_view)/urdf/dropping_box_base.urdf.xacro" />
   <!-- Instantiate quadrotor_base_macro once (has no parameters atm) -->
   <!-- model_name must be ual_${id} for ual node to find the uav -->

File: visualization/urdf/dropping_box_base.urdf.xacro (robot description, xacro)
@@ -19,21 +19,21 @@
       </inertial>
       <visual>
-      <origin xyz="0 0 0" rpy="0 0 0" />
-      <geometry>
-          <box size="0.3 0.3 0.20"/>
-      </geometry>
-      <material name="blue">
-          <color rgba="0 0 .8 1"/>
-      </material>
-    </visual>
-    <collision>
-      <origin xyz="0 0 0" rpy="0 0 0" />
-      <geometry>
-          <box size="0.3 0.3 0.20"/>
-      </geometry>
-    </collision>
-  </link>
+        <origin xyz="0 0 0" rpy="0 0 0" />
+        <geometry>
+            <box size="0.5 1 0.05"/>
+        </geometry>
+        <material name="gold">
+            <color rgba="0 1 1 1"/>
+        </material>
+      </visual>
+      <collision>
+        <origin xyz="0 0 0" rpy="0 0 0" />
+        <geometry>
+            <box size="0.5 1 0.05"/>
+        </geometry>
+        </collision>
+    </link>
     <gazebo reference="base_link_${id}">
-      <material>Gazebo/Blue</material>
+      <material>Gazebo/Gold</material>
       <turnGravityOff>false</turnGravityOff>
     </gazebo>

File: visualization/urdf/grvc_quadrotor_base.urdf.xacro (robot description, xacro)
@@ -175,5 +175,47 @@
     </gazebo>
   </xacro:macro>
-  <!-- ######################################################################## -->
+<!-- ###########################GRIPPER########################################### -->
+  <xacro:macro name="gripper" params="id">
+    <link name="gripper_pole_${id}">
+      <inertial>
+        <mass value="0.000" />
+        <origin xyz="0 0 0" rpy="0 0 0" />
+        <inertia ixx="0.00000000" ixy="0" ixz="0" iyy="0.00000000" iyz="0" izz="0.00000000" />
+      </inertial>
+      <visual>
+        <origin xyz="0 0 0" rpy="0 0 0" />
+        <geometry>
+          <cylinder length="0.2" radius=".01"/>
+        </geometry>
+      </visual>
+      <collision>
+        <origin xyz="0 0 0" rpy="0 0 0" />
+        <geometry>
+          <cylinder length="0.2" radius=".01"/>
+        </geometry>
+      </collision>
+    </link>
+    <link name="left_gripper_${id}">
+        <visual>
+          <origin rpy="0.0 0 0" xyz="0 0 0"/>
+          <geometry>
+            <mesh filename="package://pr2_description/meshes/gripper_v0/l_finger.dae"/>
+          </geometry>
+        </visual>
+    </link>
+    <joint name="left_gripper_joint_${id}" type="fixed">
+        <!--axis xyz="0 0 1"/>
+        <limit effort="1000.0" lower="0.0" upper="0.548" velocity="0.5"/-->
+        <origin rpy="0 0 0" xyz="0.2 0.01 0"/>
+        <parent link="gripper_pole_${id}"/>
+        <child link="left_gripper_${id}"/>
+    </joint>
+    <joint name="gripper_${id}_joint" type="fixed">
+      <origin xyz="0 0 -0.065" rpy="0 0 0"/>
+      <parent link="base_link_${id}"/>
+      <child link="gripper_pole_${id}"/>
+    </joint>
+  </xacro:macro>
+  <!-- ########################UAV################################################ -->
   <!-- Main quadrotor link -->
   <xacro:macro name="quadrotor_base_macro" params="id model_name">
@@ -205,4 +247,5 @@
     <xacro:generic_camera  id="${id}" />
     <xacro:sonar_sensor id="${id}" />
+    <xacro:gripper id="${id}" />
     <gazebo reference="base_link_${id}">
       <turnGravityOff>false</turnGravityOff>

File: visualization/urdf/object_black_cylinder_base.urdf.xacro (robot description, xacro)
@@ -14,7 +14,7 @@
   <link name="base_link_${id}">
     <inertial>
-      <mass value="0.1" />
+      <mass value="0.01" />
       <origin xyz="0 0 0.0" />
-      <inertia ixx="0.01152" ixy="0.0" ixz="0.0" iyy="0.01152" iyz="0.0" izz="0.0218" />
+      <inertia ixx="0.01" ixy="0.0" ixz="0.0" iyy="0.01" iyz="0.0" izz="0.01" />
     </inertial>
     <visual>

Commit message: Delete old dependencies hector quadrotor in big objects & drop_box

File: visualization/urdf/dropping_box.urdf.xacro (robot description, xacro)
@@ -8,5 +8,5 @@
 -->
 <robot name="grvc_quadrotor" xmlns:xacro="http://ros.org/wiki/xacro">
-  <xacro:arg name="model_name" default="object_blue_box_mov"/>
+  <xacro:arg name="model_name" default="drop_box"/>
   <xacro:arg name="id" default="1"/>
   <!-- Included URDF Files -->
@@ -14,4 +14,4 @@
   <!-- Instantiate quadrotor_base_macro once (has no parameters atm) -->
   <!-- model_name must be ual_${id} for ual node to find the uav -->
-  <xacro:quadrotor_base_macro id="$(arg id)" model_name="$(arg model_name)"/>
+  <xacro:drop_box id="$(arg id)" model_name="$(arg model_name)"/>
 </robot>

File: visualization/urdf/dropping_box_base.urdf.xacro (robot description, xacro)
@@ -1,15 +1,6 @@
 <?xml version="1.0"?>
-<!--
-The MIT License (MIT)
-Copyright (c) 2016 GRVC University of Seville
-Permission is hereby granted, free of charge, to any person obtaining a copy of this software and associated documentation files (the "Software"), to deal in the Software without restriction, including without limitation the rights to use, copy, modify, merge, publish, distribute, sublicense, and/or sell copies of the Software, and to permit persons to whom the Software is furnished to do so, subject to the following conditions:
-The above copyright notice and this permission notice shall be included in all copies or substantial portions of the Software.
-THE SOFTWARE IS PROVIDED "AS IS", WITHOUT WARRANTY OF ANY KIND, EXPRESS OR IMPLIED, INCLUDING BUT NOT LIMITED TO THE WARRANTIES OF MERCHANTABILITY, FITNESS FOR A PARTICULAR PURPOSE AND NONINFRINGEMENT. IN NO EVENT SHALL THE AUTHORS OR COPYRIGHT HOLDERS BE LIABLE FOR ANY CLAIM, DAMAGES OR OTHER LIABILITY, WHETHER IN AN ACTION OF CONTRACT, TORT OR OTHERWISE, ARISING FROM, OUT OF OR IN CONNECTION WITH THE SOFTWARE OR THE USE OR OTHER DEALINGS IN THE SOFTWARE.
--->
 <robot xmlns:xacro="http://ros.org/wiki/xacro">
-<xacro:include filename="$(find grvc_quadrotor_gazebo)/urdf/quadrotor_plugins.urdf.xacro" />
-<!--#####################################################################################-->
 <!-- Main quadrotor link -->
-<xacro:macro name="quadrotor_base_macro" params="id model_name">
+<xacro:macro name="drop_box" params="id model_name">
   <link name="base_link_${id}">
     <inertial>
@@ -31,6 +22,4 @@
     </collision>
   </link>
-    <!-- Gazebo Plugins -->
-    <xacro:quadrotor_plugins model_name="${model_name}" base_link="base_link_${id}"/>
   </xacro:macro>
 </robot>

File: visualization/urdf/object_big.urdf.xacro (robot description, xacro)
@@ -8,5 +8,5 @@
 -->
 <robot name="grvc_quadrotor" xmlns:xacro="http://ros.org/wiki/xacro">
-  <xacro:arg name="model_name" default="object_blue_cylinder_mov"/>
+  <xacro:arg name="model_name" default="object_big_object"/>
   <xacro:arg name="id" default="1"/>
   <!-- Included URDF Files -->
@@ -14,4 +14,4 @@
   <!-- Instantiate quadrotor_base_macro once (has no parameters atm) -->
   <!-- model_name must be ual_${id} for ual node to find the uav -->
-  <xacro:quadrotor_base_macro id="$(arg id)" model_name="$(arg model_name)"/>
+  <xacro:big_object id="$(arg id)" model_name="$(arg model_name)"/>
 </robot>

File: visualization/urdf/object_big_base.urdf.xacro (robot description, xacro)
@@ -1,15 +1,6 @@
 <?xml version="1.0"?>
-<!--
-The MIT License (MIT)
-Copyright (c) 2016 GRVC University of Seville
-Permission is hereby granted, free of charge, to any person obtaining a copy of this software and associated documentation files (the "Software"), to deal in the Software without restriction, including without limitation the rights to use, copy, modify, merge, publish, distribute, sublicense, and/or sell copies of the Software, and to permit persons to whom the Software is furnished to do so, subject to the following conditions:
-The above copyright notice and this permission notice shall be included in all copies or substantial portions of the Software.
-THE SOFTWARE IS PROVIDED "AS IS", WITHOUT WARRANTY OF ANY KIND, EXPRESS OR IMPLIED, INCLUDING BUT NOT LIMITED TO THE WARRANTIES OF MERCHANTABILITY, FITNESS FOR A PARTICULAR PURPOSE AND NONINFRINGEMENT. IN NO EVENT SHALL THE AUTHORS OR COPYRIGHT HOLDERS BE LIABLE FOR ANY CLAIM, DAMAGES OR OTHER LIABILITY, WHETHER IN AN ACTION OF CONTRACT, TORT OR OTHERWISE, ARISING FROM, OUT OF OR IN CONNECTION WITH THE SOFTWARE OR THE USE OR OTHER DEALINGS IN THE SOFTWARE.
--->
 <robot xmlns:xacro="http://ros.org/wiki/xacro">
-<xacro:include filename="$(find grvc_quadrotor_gazebo)/urdf/quadrotor_plugins.urdf.xacro" />
-<!--#####################################################################################-->
   <!-- Main object link -->
-  <xacro:macro name="quadrotor_base_macro" params="id model_name">
+  <xacro:macro name="big_object" params="id model_name">
     <link name="base_link_${id}">
       <inertial>
@@ -38,6 +29,4 @@
       <turnGravityOff>false</turnGravityOff>
     </gazebo>
-    <!-- Gazebo Plugins -->
-    <xacro:quadrotor_plugins model_name="${model_name}" base_link="base_link_${id}"/>
   </xacro:macro>
 </robot>
