Commit message: New dimensions for big object MBZIRC

File: visualization/urdf/object_big_base.urdf.xacro (robot description, xacro)
@@ -12,5 +12,5 @@
       <origin xyz="0 0 0" rpy="0 0 1.57" />
       <geometry>
-          <box size="2 0.2 0.2"/>
+          <box size="2 0.15 0.15"/>
       </geometry>
       <material name="black">
@@ -21,5 +21,5 @@
       <origin xyz="0 0 0" rpy="0 0 0" />
       <geometry>
-          <box size="2 0.2 0.2"/>
+          <box size="2 0.15 0.15"/>
       </geometry>
     </collision>
